Commit message: edit example

File: urdf-and-simulation/example/skid_steer_robot/urdf/skid_robot.urdf.xacro (robot description, xacro)
@@ -46,5 +46,5 @@
           <cylinder radius="0.06" length="0.02"/>
       </geometry>
-      <origin rpy="0 0 0"/>
+      <origin rpy="1.5708 0 0"/>
       <material name="">
         <color rgba="0.0 0.0 0.0 1.0"/>
@@ -55,5 +55,5 @@
           <cylinder radius="0.06" length="0.02"/>
       </geometry>
-      <origin rpy="0 0 0"/>
+      <origin rpy="1.5708 0 0"/>
   </collision>
   <inertial>
@@ -67,6 +67,6 @@
   <parent link="base_link"/>
   <child link="front_right_wheel"/>
-  <origin xyz="0.16 -0.16 0.05" rpy="0 1.5708 1.5708"/>
-  <axis xyz="0 0 1"/>
+  <origin xyz="0.16 -0.16 0.05" rpy="0 0 0"/>
+  <axis xyz="0 1 0"/>
 </joint>
   <!-- Front Left Wheel Link -->
@@ -76,5 +76,5 @@
             <cylinder radius="0.06" length="0.02"/>
         </geometry>
-        <origin rpy="0 0 0"/>
+        <origin rpy="1.5708 0 0"/>
         <material name="">
           <color rgba="0.0 0.0 0.0 1.0"/>
@@ -85,5 +85,5 @@
             <cylinder radius="0.06" length="0.02"/>
         </geometry>
-        <origin rpy="0 0 0"/>
+        <origin rpy="1.5708 0 0"/>
     </collision>
     <inertial>
@@ -96,6 +96,6 @@
     <parent link="base_link"/>
     <child link="front_left_wheel"/>
-    <origin xyz="0.16 0.16 0.05" rpy="0 1.5708 1.5708"/>
-    <axis xyz="0 0 1"/>
+    <origin xyz="0.16 0.16 0.05" rpy="0 0 0"/>
+    <axis xyz="0 1 0"/>
   </joint>
    <!-- Rear Right Wheel Link -->
@@ -105,5 +105,5 @@
             <cylinder radius="0.06" length="0.02"/>
         </geometry>
-        <origin rpy="0 0 0"/>
+        <origin rpy="1.5708 0 0"/>
         <material name="">
           <color rgba="0.0 0.0 0.0 1.0"/>
@@ -114,5 +114,5 @@
             <cylinder radius="0.06" length="0.02"/>
         </geometry>
-        <origin rpy="0 0 0"/>
+        <origin rpy="1.5708 0 0"/>
     </collision>
     <inertial>
@@ -125,6 +125,6 @@
     <parent link="base_link"/>
     <child link="rear_right_wheel"/>
-    <origin xyz="-0.16 -0.16 0.05" rpy="0 1.5708 1.5708"/>
-    <axis xyz="0 0 1"/>
+    <origin xyz="-0.16 -0.16 0.05" rpy="0 0 0"/>
+    <axis xyz="0 1 0"/>
   </joint>
    <!-- Rear Left Wheel Link -->
@@ -134,5 +134,5 @@
             <cylinder radius="0.06" length="0.02"/>
         </geometry>
-        <origin rpy="0 0 0"/>
+        <origin rpy="1.5708 0 0"/>
         <material name="">
           <color rgba="0.0 0.0 0.0 1.0"/>
@@ -143,5 +143,5 @@
             <cylinder radius="0.06" length="0.02"/>
         </geometry>
-        <origin rpy="0 0 0"/>
+        <origin rpy="1.5708 0 0"/>
     </collision>
     <inertial>
@@ -154,6 +154,6 @@
     <parent link="base_link"/>
     <child link="rear_left_wheel"/>
-    <origin xyz="-0.16 0.16 0.05" rpy="0 1.5708 1.5708"/>
-    <axis xyz="0 0 1"/>
+    <origin xyz="-0.16 0.16 0.05" rpy="0 0 0"/>
+    <axis xyz="0 1 0"/>
   </joint>
 <xacro:sensor_d435 parent="base_link" use_nominal_extrinsics="true">
